Commit message: added gazebo simulation

File: install/mycobot_moveit_config_new/share/mycobot_moveit_config_new/config/mycobot_280.ros2_control.xacro (robot description, xacro)
@@ -2,9 +2,9 @@
 <robot xmlns:xacro="http://www.ros.org/wiki/xacro">
     <xacro:macro name="mycobot_280_ros2_control" params="name initial_positions_file">
-        <xacro:property name="initial_positions" value="${load_yaml(initial_positions_file)['initial_positions']}"/>
+        <xacro:property name="initial_positions" value="${xacro.load_yaml(initial_positions_file)['initial_positions']}"/>
         <ros2_control name="${name}" type="system">
             <hardware>
                 <!-- By default, set up controllers for simulation. This won't work on real hardware -->
-                <plugin>mock_components/GenericSystem</plugin>
+                <plugin>gazebo_ros2_control/GazeboSystem</plugin>
             </hardware>
             <joint name="link1_to_link2">

File: install/mycobot_moveit_config_new/share/mycobot_moveit_config_new/config/mycobot_280.urdf.xacro (robot description, xacro)
@@ -6,4 +6,11 @@
     <!-- Import control_xacro -->
     <xacro:include filename="mycobot_280.ros2_control.xacro" />
-    <xacro:mycobot_280_ros2_control name="FakeSystem" initial_positions_file="$(arg initial_positions_file)"/>
+    <!-- Instantiate the ros2_control xacro to generate the <ros2_control> tag -->
+    <xacro:mycobot_280_ros2_control name="GazeboSystem" initial_positions_file="$(arg initial_positions_file)"/>
+    <!-- Gazebo Classic Plugin for ros2_control -->
+    <gazebo>
+        <plugin filename="libgazebo_ros2_control.so" name="gazebo_ros2_control">
+            <parameters>$(find mycobot_moveit_config_new)/config/ros2_controllers.yaml</parameters>
+        </plugin>
+    </gazebo>
 </robot>
